File: pcb/keypad/keypad_keys.kicad_sch (KiCad schematic)
At the start: 50 parts, among them SW1 Y=, SW10 ON, SW11 WINDOW, SW12 MODE, SW13 XTTN, SW14 APPS, SW15 SIN, SW16 COMMA, SW17 7, SW18 4, SW19 1, SW2 2ND, SW20 0, SW21 ZOOM, SW22 DEL, SW23 STAT, SW24 PRGM, SW25 COS, SW26 LBRACKET, SW27 8, SW28 5, SW29 2, SW3 ALPHA, SW30 DOT, SW31 L, SW32 TRACE, SW33 VARS, SW34 TAN, SW35 RBRACKET, SW36 9, SW37 6, SW38 3, SW39 NEG, SW4 MATH, SW40 U, SW41 D, SW42 GRAPH, SW43 CLEAR, SW44 HAT, SW45 DIV, SW46 MUL, SW47 SUB, SW48 ADD, SW49 ENTER, SW5 X-1, SW50 R, SW6 X2, SW7 LOG, SW8 LN, SW9 STO

Commit message: Keypad Layout Done V1
Parts:
- SW10: footprint keypad:key2 -> keypad:key3
Changed lines of the file:
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@@
     (property "Reference" "SW10" (id 0) (at 43.18 165.1 0))
     (property "Value" "ON" (id 1) (at 43.18 167.64 0))
-    (property "Footprint" "keypad:key2" (id 2) (at 43.18 172.72 0)
+    (property "Footprint" "keypad:key3" (id 2) (at 43.18 172.72 0)
       (effects (font (size 1.27 1.27)) hide)
     )

Commit message: Keypad bugfix, pulling in submodules
Connections:
- net KR7: now reaches SW13.2, SW22.2, SW23.2, SW3.2
