File: pcb/mainboard/keypad.kicad_sch (KiCad schematic)
At the start: 7 parts, among them U201 MIMX8MN6DVTJZAA

Commit message: Routing mainboard in progress, schematics fixes
Parts:
- removed J?: Conn_01x40_MountingPin, Connector_FFC-FPC:TE_4-1734839-0_1x40-1MP_P0.5mm_Horizontal, symbol Connector_Generic_MountingPin:Conn_01x40_MountingPin
- removed R603, R604: 4.7K, Resistor_SMD:R_0402_1005Metric, symbol Device:R
- added J601: Conn_01x12_MountingPin, Connector_FFC-FPC:TE_1-1734839-2_1x12-1MP_P0.5mm_Horizontal, symbol Connector_Generic_MountingPin:Conn_01x12_MountingPin
- added J602: Conn_01x24_MountingPin, Connector_FFC-FPC:TE_2-1734839-4_1x24-1MP_P0.5mm_Horizontal, symbol Connector_Generic_MountingPin:Conn_01x24_MountingPin
- gave numbers to parts that had none: 1
Connections:
- net +1V8: now also J601.2 (Pin_2)
- net +3V3: now also J602.1 (Pin_1)
- net BATP: now also J602.2 (Pin_2), J602.3 (Pin_3), J602.4 (Pin_4), J602.5 (Pin_5)
- net GND: now also J601.1 (Pin_1), J601.8 (Pin_8), J601.MP (MountPin), J602.24 (Pin_24), J602.6 (Pin_6), J602.7 (Pin_7), J602.8 (Pin_8), J602.MP (MountPin)
- net JTAG_TCK: now also J601.6 (Pin_6)
- net JTAG_TDI: now also J601.4 (Pin_4)
- net JTAG_TDO: now also J601.5 (Pin_5)
- net JTAG_TMS: now also J601.7 (Pin_7)
- net KC0: now also J602.16 (Pin_16)
- net KC1: now also J602.15 (Pin_15)
- net KC2: now also J602.14 (Pin_14)
- net KC3: now also J602.13 (Pin_13)
- net KC4: now also J602.12 (Pin_12)
- net KC5: now also J602.11 (Pin_11)
- net KC6: now also J602.10 (Pin_10)
- net KR0: now also J602.23 (Pin_23)
- net KR1: now also J602.22 (Pin_22)
- net KR2: now also J602.21 (Pin_21)
- net KR3: now also J602.20 (Pin_20)
- net KR4: now also J602.19 (Pin_19)
- net KR5: now also J602.18 (Pin_18)
- net KR6: now also J602.17 (Pin_17)
- net LCD_RST: now also U201.AF14 (GPIO1_IO01); no longer U201.AF11 (GPIO1_IO07)
- net ONOFF: now also J602.9 (Pin_9)
- net UART2_RXD: now also J601.9 (Pin_9)
- net UART2_TXD: now also J601.11 (Pin_11)
- net UART4_RXD: now also J601.10 (Pin_10)
- net UART4_TXD: now also J601.12 (Pin_12)
- net TASKSEL: now reaches U201.AG24 (ENET_TXC)
- net at D601.1 (K): now also J601.3 (Pin_3)
- net I2C3_SCL: no longer names the net of U201.E10 (I2C3_SCL)
- net I2C3_SDA: no longer names the net of U201.F10 (I2C3_SDA)
- no-connect marks 23 -> 22

Commit message: Keypad bugfix, pulling in submodules
Connections:
- net GND: no longer J602.8 (Pin_8)
- net KC7: now reaches U201.AB9 (GPIO1_IO15)
- net KC7: now also J602.8 (Pin_8)
- no-connect marks 22 -> 27
