File: pcb/mainboard/lcd.kicad_sch (KiCad schematic)
At the start: 4 parts, among them J501 Conn_02x15_Row_Letter_First_M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, U501 TPS65631W

Commit message: Working on mainboard schematics
Parts:
- removed U501: TPS65631W, symbol symbols:TPS65631W
- added C? (x6): 10uF, Capacitor_SMD:C_0603_1608Metric, symbol Device:C
- added C? (x2): 100nF, Capacitor_SMD:C_0201_0603Metric, symbol Device:C
- added L?: 10uH, Inductor_SMD:L_1008_2520Metric, symbol Device:L
- added L? (x2): 4.7uH, Inductor_SMD:L_1008_2520Metric, symbol Device:L
- added R? (x2): 0, Resistor_SMD:R_0402_1005Metric, symbol Device:R
- added R? (x2): DNP, Resistor_SMD:R_0402_1005Metric, symbol Device:R
- added U?: TPS65632, Package_DFN_QFN:QFN-16-1EP_3x3mm_P0.5mm_EP1.7x1.7mm, symbol symbols:TPS65632
Connections:
- net GND: now also C?.1, C?.1, C?.1, C?.1, C?.1, C?.1, C?.1, C?.1, L?.2, U?.14 (PGND2), U?.17 (EP), U?.2 (PGND1), U?.5 (SELP2), U?.7 (AGND)
- net SWIRE: now reaches J501.b11 (Pin_b11)
- net SWIRE: now also R?.2
- net OLED_EN: now reaches J501.b12 (Pin_b12)
- net OLED_EN: now also R?.2
- net VPOS: now reaches J501.b2 (Pin_b2)
- net VPOS: now also J501.b3 (Pin_b3), C?.2, U?.3 (OUTP1), U?.4 (FBS)
- net VNEG: now reaches J501.b4 (Pin_b4)
- net VNEG: now also J501.b5 (Pin_b5), C?.2, U?.10 (OUTN)
- net AVDD: now reaches J501.b6 (Pin_b6)
- net AVDD: now also C?.2, U?.13 (OUTP2)
- net +1V8: now reaches J501.b8 (Pin_b8)
- net +3V3: now reaches J501.b9 (Pin_b9)
- new net: L?.2, U?.15 (SWP2)
- new net: L?.2, U?.1 (SWP1)
- new net: R?.1, R?.1, U?.9 (CTRL)
- new net: C?.2, U?.6 (CT)
- new net: R?.1, R?.1, U?.8 (EN)
- new net: L?.1, U?.11 (SWN)
- new net +BATT: C?.2, C?.2, C?.2, C?.2, L?.1, L?.1, U?.12 (PVIN), U?.16 (AVIN)
- new net AVDD_EN: R?.2
- new net VNEG_CTRL: R?.2
- no-connect marks 0 -> 20
Other:
- moved on the sheet: J501

Commit message: Mainboard schematics WIP
Parts:
- removed J501: Conn_02x15_Row_Letter_First_MountingPin, symbol Connector_Generic_MountingPin:Conn_02x15_Row_Letter_First_MountingPin
- added J501: Conn_02x15_Odd_Even_MountingPin, footprint:505270-3012, symbol Connector_Generic_MountingPin:Conn_02x15_Odd_Even_MountingPin
- gave numbers to parts that had none: 17
Connections:
- net +1V8: now also J501.16 (Pin_16)
- net +3V3: now also J501.18 (Pin_18)
- net AVDD: now also J501.12 (Pin_12)
- net GND: now also J501.14 (Pin_14), J501.15 (Pin_15), J501.2 (Pin_2), J501.20 (Pin_20), J501.21 (Pin_21), J501.27 (Pin_27), J501.9 (Pin_9), J501.MP (MountPin)
- net LCD_RST: now also J501.30 (Pin_30)
- net MIPI_CKN: now also J501.17 (Pin_17)
- net MIPI_CKP: now also J501.19 (Pin_19)
- net MIPI_D0N: now also J501.23 (Pin_23)
- net MIPI_D0P: now also J501.25 (Pin_25)
- net MIPI_D1N: now also J501.11 (Pin_11)
- net MIPI_D1P: now also J501.13 (Pin_13)
- net OLED_EN: now also J501.24 (Pin_24)
- net SWIRE: now also J501.22 (Pin_22)
- net VNEG: now also J501.10 (Pin_10), J501.8 (Pin_8)
- net VPOS: now also J501.4 (Pin_4), J501.6 (Pin_6)
