File: pcb/mainboard/pcb.kicad_pcb (KiCad board)
At the start: 4 copper layers, 67.2 x 58.2 mm, 224 parts, among them J401 AudioJack3, J501 Conn_02x15_Odd_Even_MountingP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, J601 Conn_01x12_MountingPin, J602 Conn_01x24_MountingPin, J801 USB_B_Mini, SW101 SW_Push, SW201 SW_Push, U101 PCA9450BHN, U102 BQ27441-G1, U103 BQ24072RGT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

Commit message: Keypad bugfix, pulling in submodules
Parts:
- moved C245 0.08 mm to (158.2, 103.3)
- renumbered R208 to R804
Connections:
- J602 pad 8: GND -> KC7
- U201 pad AB9: unconnected-(U201-PadAB9) -> KC7
Routing:
- net KC7: track 0.00 -> 29.8 mm, vias 0 -> 2
- net GND: track 225.7 -> 224.4 mm, vias 284 -> 283
- net KC1: track 31.3 -> 31.8 mm
