File: pcb/mainboard/pcb.kicad_sch (KiCad schematic)
At the start: 0 parts

Commit message: Working on mainboard schematics
Other:
- note added: "Display"
- note added: "Processor"
- note removed: "LCD"
- note removed: "MCU"
