File: pcb/mainboard/power.kicad_sch (KiCad schematic)
At the start: 0 parts

Commit message: Working on mainboard schematics
Parts:
- added C? (x4): 4.7uF, Capacitor_SMD:C_0402_1005Metric, symbol Device:C
- added C? (x4): 10uF, Capacitor_SMD:C_0603_1608Metric, symbol Device:C
- added C? (x2): 18pF, Capacitor_SMD:C_0402_1005Metric, symbol Device:C
- added C?: 2.2uF, Capacitor_SMD:C_0402_1005Metric, symbol Device:C
- added C? (x7): 1uF, Capacitor_SMD:C_0201_0603Metric, symbol Device:C
- added C? (x7): 22uF, Capacitor_SMD:C_0603_1608Metric, symbol Device:C
- added C? (x4): 1uF, Capacitor_SMD:C_0402_1005Metric, symbol Device:C
- added L? (x5): 0.47uH, Inductor_SMD:L_1008_2520Metric, symbol Device:L
- added R? (x2): 10K, Resistor_SMD:R_0402_1005Metric, symbol Device:R
- added R?: 0, Resistor_SMD:R_0402_1005Metric, symbol Device:R
- added R?: 0.01/1%, symbol Device:R
- added R?: 1K, Resistor_SMD:R_0402_1005Metric, symbol Device:R
- added R?: 2K, Resistor_SMD:R_0402_1005Metric, symbol Device:R
- added SW?: SW_Push, symbol Switch:SW_Push
- added U?: BQ24072RGT, Package_DFN_QFN:VQFN-16-1EP_3x3mm_P0.5mm_EP1.6x1.6mm, symbol Battery_Management:BQ24072RGT
- added U? (x2): PCA9450BHN, symbol symbols:PCA9450BHN
- added U?: PCA9450BHN, footprint:QFN-56_EP_7x7_Pitch0.4mm, symbol symbols:PCA9450BHN
- added U?: BQ27441-G1, Package_SON:Texas_S-PDSO-N12, symbol Battery_Management:BQ27441-G1
- added Y?: 32.768K, Crystal:Crystal_SMD_TXC_9HT11-2Pin_2.0x1.2mm_HandSoldering, symbol Device:Crystal
Connections:
- new net: R?.1, U?.10 (BIN)
- new net: L?.1, U?.45 (LX2), U?.46 (LX2)
- new net: C?.2, U?.10 (XTAL_IN), Y?.1
- new net: R?.1, U?.12 (ILIM)
- new net: R?.1, U?.16 (ISET)
- new net: C?.2, U?.11 (XTAL_OUT), Y?.2
- new net: C?.2, U?.4 (VINT)
- new net: SW?.2, U?.8 (PMIC_RST_B)
- new net: L?.1, U?.50 (LX6), U?.51 (LX6)
- new net: L?.1, U?.15 (LX5)
- new net: R?.2, U?.30 (R_SNSP3_CFG)
- new net: R?.2, U?.12 (GPOUT)
- new net: L?.1, U?.19 (LX4), U?.20 (LX4)
- new net: L?.1, U?.36 (LX1), U?.37 (LX1)
- new net: C?.2, U?.5 (VDD)
- new net +1V1: C?.2, L?.2, U?.52 (BUCK6FB)
- new net +1V2: C?.2, U?.1 (LDO4)
- new net +1V8: C?.2, L?.2, R?.1, U?.14 (BUCK5FB)
- new net +1V8A: C?.2, U?.54 (LDO3)
- new net +3V3: C?.2, C?.2, L?.2, U?.21 (BUCK4FB), U?.22 (SWIN)
- new net +BATT: C?.2, C?.2, C?.2, C?.2, C?.2, C?.2, C?.2, C?.2, C?.2, R?.1, U?.10 (OUT), U?.11 (OUT), U?.16 (INB45), U?.17 (INB45), U?.33 (INB13), U?.34 (INB13), U?.47 (INB26), U?.48 (INB26), U?.49 (INB26), U?.53 (VSYS), U?.56 (INL1)
- new net +SD: C?.2, U?.23 (SWOUT)
- new net +VCCIO_SD: C?.2, U?.55 (LDO5)
- new net BATP: C?.2, R?.1, U?.6 (BAT), U?.8 (SRP)
- new net BAT_CHRG: U?.9 (~{CHG})
- new net BAT_FG: R?.2, U?.2 (BAT), U?.3 (BAT), U?.7 (SRN)
- new net BAT_TS: U?.1 (TS)
- new net CLK_32K_OUT: U?.7 (CLK_32K_OUT)
- new net GND: C?.1, C?.1, C?.1, C?.1, C?.1, C?.1, C?.1, C?.1, C?.1, C?.1, C?.1, C?.1, C?.1, C?.1, C?.1, C?.1, C?.1, C?.1, C?.1, C?.1, C?.1, C?.1, C?.1, C?.1, C?.1, C?.1, C?.1, C?.1, C?.1, R?.2, R?.2, R?.2, SW?.1, U?.13 (PAD), U?.14 (TMR), U?.15 (TD), U?.17 (VSS), U?.3 (VSS), U?.4 (~{CE}), U?.43 (BUCK_AGND), U?.5 (AGND), U?.57 (EPAD), U?.6 (EN1), U?.8 (VSS)
- new net I2C1_SCL: U?.2 (SCL), U?.41 (SCL)
- new net I2C1_SDA: U?.1 (SDA), U?.42 (SDA)
- new net PMIC_INT: U?.13 (IRQ_B)
- new net PMIC_ON_REQ: U?.39 (PMIC_ON_REQ)
- new net PMIC_STBY_REQ: U?.40 (PMIC_STBY_REQ)
- new net POR_B: U?.9 (POR_B)
- new net RTC_0P8: C?.2, U?.2 (LDO2)
- new net RTC_1P8: C?.2, U?.3 (LDO1)
- new net RTC_RESET_B: U?.6 (RTC_RESET_B)
- new net SD2_VSEL: U?.29 (SD_VSEL)
- new net SD_NRST: U?.12 (SW_EN)
- new net VBUS: C?.2, U?.13 (IN)
- new net VDD_ARM: C?.2, C?.2, L?.2, U?.44 (R_SNSP2)
- new net VDD_SOC: C?.2, C?.2, L?.2, U?.38 (R_SNSP1)
- new net WDOG_B: U?.28 (WDOG_B)
- no-connect marks 0 -> 3

Commit message: Mainboard schematics WIP
Parts:
- gave numbers to parts that had none: 45

Commit message: Draft motherboard schematics for r0.0 layout
Parts:
- L101, L102, L103, L104, L105: value 0.47uH -> 470nH
- R102: footprint (none) -> Resistor_SMD:R_0603_1608Metric
- SW101: footprint (none) -> Button_Switch_SMD:SW_SPST_SKQG_WithStem
- U101: footprint (none) -> footprint:QFN-56_EP_7x7_Pitch0.4mm
Changed lines of the file:
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@@
     (in_bom yes) (on_board yes)
     (property "Reference" "L101" (id 0) (at 87.63 35.56 90))
-    (property "Value" "0.47uH" (id 1) (at 87.63 38.1 90))
+    (property "Value" "470nH" (id 1) (at 87.63 38.1 90))
     (property "Footprint" "Inductor_SMD:L_1008_2520Metric" (id 2) (at 87.63 40.64 0)
       (effects (font (size 1.27 1.27)) hide)
@@
     (pin "2")
   )
-  (symbol (lib_id "symbols:PCA9450BHN") (at 246.38 22.86 0) (unit 3)
+  (symbol (lib_name "PCA9450BHN_2") (lib_id "symbols:PCA9450BHN") (at 246.38 22.86 0) (unit 3)
     (in_bom yes) (on_board yes)
     (property "Reference" "U101" (id 0) (at 238.76 33.02 0)
@@
       (effects (font (size 1.27 1.27)) (justify left))
     )
-    (property "Footprint" "" (id 2) (at 246.38 22.86 0)
+    (property "Footprint" "footprint:QFN-56_EP_7x7_Pitch0.4mm" (id 2) (at 246.38 22.86 0)
       (effects (font (size 1.27 1.27)) hide)
     )
@@
     (in_bom yes) (on_board yes)
     (property "Reference" "L105" (id 0) (at 87.63 111.76 90))
-    (property "Value" "0.47uH" (id 1) (at 87.63 114.3 90))
+    (property "Value" "470nH" (id 1) (at 87.63 114.3 90))
     (property "Footprint" "Inductor_SMD:L_1008_2520Metric" (id 2) (at 87.63 116.84 0)
       (effects (font (size 1.27 1.27)) hide)
@@
     (in_bom yes) (on_board yes)
     (property "Reference" "L104" (id 0) (at 87.63 96.52 90))
-    (property "Value" "0.47uH" (id 1) (at 87.63 99.06 90))
+    (property "Value" "470nH" (id 1) (at 87.63 99.06 90))
     (property "Footprint" "Inductor_SMD:L_1008_2520Metric" (id 2) (at 87.63 101.6 0)
       (effects (font (size 1.27 1.27)) hide)
@@
     (property "Reference" "R102" (id 0) (at 151.13 118.11 90))
     (property "Value" "0.01/1%" (id 1) (at 151.13 120.65 90))
-    (property "Footprint" "" (id 2) (at 151.13 126.238 90)
+    (property "Footprint" "Resistor_SMD:R_0603_1608Metric" (id 2) (at 151.13 126.238 90)
       (effects (font (size 1.27 1.27)) hide)
     )
@@
     (property "Reference" "SW101" (id 0) (at 226.06 38.1 0))
     (property "Value" "SW_Push" (id 1) (at 226.06 40.64 0))
-    (property "Footprint" "" (id 2) (at 226.06 40.64 0)
+    (property "Footprint" "Button_Switch_SMD:SW_SPST_SKQG_WithStem" (id 2) (at 226.06 40.64 0)
       (effects (font (size 1.27 1.27)) hide)
     )
@@
     (in_bom yes) (on_board yes)
     (property "Reference" "L103" (id 0) (at 87.63 81.28 90))
-    (property "Value" "0.47uH" (id 1) (at 87.63 83.82 90))
+    (property "Value" "470nH" (id 1) (at 87.63 83.82 90))
     (property "Footprint" "Inductor_SMD:L_1008_2520Metric" (id 2) (at 87.63 86.36 0)
       (effects (font (size 1.27 1.27)) hide)
@@
     (in_bom yes) (on_board yes)
     (property "Reference" "L102" (id 0) (at 87.63 50.8 90))
-    (property "Value" "0.47uH" (id 1) (at 87.63 53.34 90))
+    (property "Value" "470nH" (id 1) (at 87.63 53.34 90))
     (property "Footprint" "Inductor_SMD:L_1008_2520Metric" (id 2) (at 87.63 55.88 0)
       (effects (font (size 1.27 1.27)) hide)
@@
     (property "Reference" "U101" (id 0) (at 167.64 33.02 0))
     (property "Value" "PCA9450BHN" (id 1) (at 167.64 35.56 0))
-    (property "Footprint" "" (id 2) (at 167.64 33.02 0)
-      (effects (font (size 1.27 1.27)) hide)
-    )
+    (property "Footprint" "footprint:QFN-56_EP_7x7_Pitch0.4mm" (id 2) (at 167.64 33.02 0)
+      (effects (font (size 1.27 1.27)) hide)
+    )

Commit message: Motherboard PCB component initial placement, schematics fixes
Connections:
- net +BATT: now also U101.18 (INB45), U101.35 (INB13)
Changed lines of the file:
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@@
   (junction (at 185.42 53.34) (diameter 0) (color 0 0 0 0)
   )
+  (junction (at 45.72 58.42) (diameter 0) (color 0 0 0 0)
+  )
   (junction (at 45.72 55.88) (diameter 0) (color 0 0 0 0)
   )
@@
   )
   (junction (at 93.98 55.88) (diameter 0) (color 0 0 0 0)
+  )
+  (junction (at 45.72 88.9) (diameter 0) (color 0 0 0 0)
   )
   (junction (at 81.28 55.88) (diameter 0) (color 0 0 0 0)
@@
     (stroke (width 0) (type default) (color 0 0 0 0))
   )
+  (wire (pts (xy 45.72 58.42) (xy 45.72 71.12))
+    (stroke (width 0) (type default) (color 0 0 0 0))
+  )
   (wire (pts (xy 182.88 43.18) (xy 185.42 43.18))
     (stroke (width 0) (type default) (color 0 0 0 0))
@@
     (stroke (width 0) (type default) (color 0 0 0 0))
   )
+  (wire (pts (xy 45.72 88.9) (xy 48.26 88.9))
+    (stroke (width 0) (type default) (color 0 0 0 0))
+  )
   (wire (pts (xy 33.02 86.36) (xy 33.02 101.6))
     (stroke (width 0) (type default) (color 0 0 0 0))
@@
     (stroke (width 0) (type default) (color 0 0 0 0))
   )
-  (wire (pts (xy 45.72 55.88) (xy 45.72 71.12))
+  (wire (pts (xy 45.72 55.88) (xy 45.72 58.42))
     (stroke (width 0) (type default) (color 0 0 0 0))
   )
@@
     (stroke (width 0) (type default) (color 0 0 0 0))
   )
+  (wire (pts (xy 45.72 88.9) (xy 45.72 101.6))
+    (stroke (width 0) (type default) (color 0 0 0 0))
+  )
   (wire (pts (xy 93.98 96.52) (xy 93.98 86.36))
     (stroke (width 0) (type default) (color 0 0 0 0))
@@
   )
   (wire (pts (xy 182.88 63.5) (xy 185.42 63.5))
+    (stroke (width 0) (type default) (color 0 0 0 0))
+  )
+  (wire (pts (xy 45.72 58.42) (xy 48.26 58.42))
     (stroke (width 0) (type default) (color 0 0 0 0))
   )
@@
     (stroke (width 0) (type default) (color 0 0 0 0))
   )
-  (wire (pts (xy 45.72 86.36) (xy 45.72 101.6))
-    (stroke (width 0) (type default) (color 0 0 0 0))
-  )
+  (wire (pts (xy 45.72 86.36) (xy 45.72 88.9))
+    (stroke (width 0) (type default) (color 0 0 0 0))
+  )

Commit message: Mainboard design bug fixes
Connections:
- net +BATT: now also U103.5 (EN2)
Changed lines of the file:
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@@
+    (stroke (width 0) (type default) (color 0 0 0 0))
+  )
+  (wire (pts (xy 228.6 142.24) (xy 231.14 142.24))
     (stroke (width 0) (type default) (color 0 0 0 0))
   )
@@
       (effects (font (size 1.27 1.27)) hide)
     )
+    (pin "1")
+  )
+  (symbol (lib_id "power:+BATT") (at 228.6 142.24 90) (unit 1)
+    (in_bom yes) (on_board yes)
+    (property "Reference" "#PWR?" (id 0) (at 232.41 142.24 0)
+      (effects (font (size 1.27 1.27)) hide)
+    )
+    (property "Value" "+BATT" (id 1) (at 219.71 142.24 90)
+      (effects (font (size 1.27 1.27)) (justify right))
+    )
+    (property "Footprint" "" (id 2) (at 228.6 142.24 0)
+      (effects (font (size 1.27 1.27)) hide)
+    )
+    (property "Datasheet" "" (id 3) (at 228.6 142.24 0)
+      (effects (font (size 1.27 1.27)) hide)
+    )
